Commit message: Added UWB sensor to turtlebot3_burger. Added uwb_tag model.

File: turtlebot3_description/urdf/turtlebot3_burger.gazebo.xacro (robot description, xacro)
@@ -5,4 +5,6 @@
   <gazebo reference="base_link">
     <material>Gazebo/DarkGrey</material>
+  </gazebo>
+  <gazebo reference="uwb_link">
   </gazebo>
   <gazebo reference="wheel_left_link">
@@ -36,7 +38,11 @@
   </gazebo>
   <gazebo reference="imu_link">
+    <gravity>false</gravity>
     <sensor type="imu" name="imu">
       <always_on>true</always_on>
       <visualize>$(arg imu_visual)</visualize>
+      <update_rate>100</update_rate>
+      <gaussianNoise>0.0</gaussianNoise>
+      <pose>0 0 0 0 0 0</pose>
     </sensor>
     <material>Gazebo/FlatBlack</material>
@@ -64,5 +70,5 @@
     </plugin>
   </gazebo>
-  <gazebo>
+<!--   <gazebo>
     <plugin name="imu_plugin" filename="libgazebo_ros_imu.so">
       <alwaysOn>true</alwaysOn>
@@ -91,5 +97,5 @@
       </imu>
     </plugin>
-  </gazebo>
+  </gazebo> -->
   <gazebo reference="base_scan">
     <material>Gazebo/FlatBlack</material>
@@ -124,3 +130,85 @@
     </sensor>
   </gazebo>
+  <gazebo>
+    <plugin name='libgtec_uwb_plugin' filename='libgtec_uwb_plugin.so'>
+      <update_rate>25</update_rate>
+      <nlosSoftWallWidth>0.25</nlosSoftWallWidth>
+      <tag_z_offset>1</tag_z_offset>
+      <tag_link>base_footprint</tag_link>
+      <anchor_prefix>uwb_anchor</anchor_prefix>
+      <all_los>false</all_los>
+      <tag_id>0</tag_id>
+    </plugin>
+</gazebo>
+  <gazebo>
+    <plugin name='libgtec_tag_pos_publisher_plugin' filename='libgtec_tag_pos_publisher_plugin.so'>
+      <update_rate>40</update_rate>
+      <tag_link>base_footprint</tag_link>
+    </plugin>
+</gazebo>
+<gazebo reference="base_camera">
+<!--         <sensor name='erle_magnetometer' type='magnetometer'>
+        <update_rate>8</update_rate>
+        <always_on>1</always_on>
+        <magnetometer>
+           <x>
+            <noise type="gaussian">
+              <mean>0.0</mean>
+              <stddev>0.00000000344</stddev>
+            </noise>
+          </x>
+          <y>
+            <noise type="gaussian">
+              <mean>0.0</mean>
+              <stddev>0.00000000344</stddev>
+            </noise>
+          </y>
+          <z>
+            <noise type="gaussian">
+              <mean>0.0</mean>
+              <stddev>0.00000000344</stddev>
+            </noise>
+          </z>
+        </magnetometer>
+          <plugin name='libgtec_magnetic_distortion_plugin' filename='libgtec_magnetic_distortion_plugin.so'>
+            <field_strength>1e-5</field_strength>
+        </plugin>
+      </sensor> -->
+      <sensor type="imu" name="px4_imu">
+        <pose>0 0 0 0 -1.5707 3.1416</pose>
+        <always_on>1</always_on>
+        <update_rate>200</update_rate>
+      </sensor>
+     <sensor name="PX4Flow" type="camera">
+        <pose frame=''>0.0 0 0.0 0 1.5707 1.5707</pose>
+        <always_on>true</always_on>
+        <update_rate>20.0</update_rate>
+        <visualize>true</visualize>
+        <topic>/px4flow</topic>
+        <camera>
+          <horizontal_fov>0.088</horizontal_fov>
+          <image>
+            <width>64</width>
+            <height>64</height>
+            <format>L8</format>
+          </image>
+          <clip>
+            <near>0.1</near>
+            <far>10</far>
+          </clip>
+           <noise>
+            <type>gaussian</type>
+            <mean>0.0</mean>
+            <stddev>0.0001</stddev>
+          </noise>
+        </camera>
+       <plugin name="opticalflow_plugin" filename="libgazebo_opticalflow_plugin.so">
+            <enabled>true</enabled>
+            <robotNamespace></robotNamespace>
+            <outputRate>20</outputRate>
+            <hasGyro>true</hasGyro>
+            <gyroTopic>/px4_imu/imu</gyroTopic>
+        </plugin>
+      </sensor>
+</gazebo>
 </robot>

File: turtlebot3_description/urdf/turtlebot3_burger.urdf.xacro (robot description, xacro)
@@ -31,5 +31,12 @@
     </inertial>
   </link>
-  <joint name="wheel_left_joint" type="continuous">
+  <joint name="uwb_joint" type="fixed">
+    <parent link="base_link"/>
+    <child link="uwb_link"/>
+    <origin xyz="0 0 1" rpy="0 0 0"/>
+  </joint>
+  <link name="uwb_link">
+    </link>
+<joint name="wheel_left_joint" type="continuous">
     <parent link="base_link"/>
     <child link="wheel_left_link"/>
@@ -110,5 +117,5 @@
     <parent link="base_link"/>
     <child link="imu_link"/>
-    <origin xyz="-0.032 0 0.068" rpy="0 0 0"/>
+    <origin xyz="0 0 0" rpy="0.0 -0.0078 0"/>
   </joint>
   <link name="imu_link"/>
@@ -117,4 +124,9 @@
     <child link="base_scan"/>
     <origin xyz="-0.032 0 0.172" rpy="0 0 0"/>
+  </joint>
+  <joint name="camera_joint" type="fixed">
+    <parent link="base_link"/>
+    <child link="base_camera"/>
+    <origin xyz="1 0 5" rpy="0 1.5707 1.5707"/>
   </joint>
   <link name="base_scan">
@@ -140,3 +152,25 @@
     </inertial>
   </link>
+  <link name="base_camera">
+    <visual>
+      <origin xyz="0 0 0.0" rpy="0 0 0"/>
+      <geometry>
+        <cylinder length="0.025" radius="0.025"/>
+      </geometry>
+      <material name="dark"/>
+    </visual>
+    <collision>
+      <origin xyz="0.0 0 0.0" rpy="0 0 0"/>
+      <geometry>
+        <cylinder length="0.025" radius="0.025"/>
+      </geometry>
+    </collision>
+    <inertial>
+      <mass value="0.001" />
+      <origin xyz="0 0 0" />
+      <inertia ixx="0.001" ixy="0.0" ixz="0.0"
+               iyy="0.001" iyz="0.0"
+               izz="0.001" />
+    </inertial>
+  </link>
 </robot>
